Commit message: URDF: motor rotors on mimic joints, crank driven by output A, 4-bar closed in MuJoCo; limit-aware IK; five gaits; jump retuned

File: CapstanPedal/fullbuild_v3/urdf/capstan_quad.urdf (robot description, URDF)
Before this commit: robot capstan_quad, 21 links, 20 joints
Links:
- added link rotorA_LF, mass 0.001; visual mesh filename=meshes/rotorA_LF__magnet.stl; visual mesh filename=meshes/rotorA_LF__motor.stl
- added link rotorA_LR, mass 0.001; visual mesh filename=meshes/rotorA_LR__magnet.stl; visual mesh filename=meshes/rotorA_LR__motor.stl
- added link rotorA_RF, mass 0.001; visual mesh filename=meshes/rotorA_RF__magnet.stl; visual mesh filename=meshes/rotorA_RF__motor.stl
- added link rotorA_RR, mass 0.001; visual mesh filename=meshes/rotorA_RR__magnet.stl; visual mesh filename=meshes/rotorA_RR__motor.stl
- added link rotorB_LF, mass 0.001; visual mesh filename=meshes/rotorB_LF__magnet.stl; visual mesh filename=meshes/rotorB_LF__motor.stl
- added link rotorB_LR, mass 0.001; visual mesh filename=meshes/rotorB_LR__magnet.stl; visual mesh filename=meshes/rotorB_LR__motor.stl
- added link rotorB_RF, mass 0.001; visual mesh filename=meshes/rotorB_RF__magnet.stl; visual mesh filename=meshes/rotorB_RF__motor.stl
- added link rotorB_RR, mass 0.001; visual mesh filename=meshes/rotorB_RR__magnet.stl; visual mesh filename=meshes/rotorB_RR__motor.stl
- added link rotorC_LF, mass 0.001; visual mesh filename=meshes/rotorC_LF__magnet.stl; visual mesh filename=meshes/rotorC_LF__motor.stl
- added link rotorC_LR, mass 0.001; visual mesh filename=meshes/rotorC_LR__magnet.stl; visual mesh filename=meshes/rotorC_LR__motor.stl
- added link rotorC_RF, mass 0.001; visual mesh filename=meshes/rotorC_RF__magnet.stl; visual mesh filename=meshes/rotorC_RF__motor.stl
- added link rotorC_RR, mass 0.001; visual mesh filename=meshes/rotorC_RR__magnet.stl; visual mesh filename=meshes/rotorC_RR__motor.stl
- link pod_LF: geometry collision box size=0.26 0.10 0.17; visual mesh filename=meshes/pod_LF__black.stl
- link pod_LR: geometry collision box size=0.26 0.10 0.17; visual mesh filename=meshes/pod_LR__black.stl
- link pod_RF: geometry collision box size=0.26 0.10 0.17; visual mesh filename=meshes/pod_RF__black.stl
- link pod_RR: geometry collision box size=0.26 0.10 0.17; visual mesh filename=meshes/pod_RR__black.stl
- link torso: geometry collision box size=0.69 0.26 0.22; visual mesh filename=meshes/torso__black.stl
Joints:
- added joint LF_rotorA: type revolute, parent pod_LF, child rotorA_LF, origin xyz=-0.04675 0.00000 0.06000, axis 0 1 0, limit lower=-174.53293 upper=174.53293 effort=3.5 velocity=210, mimic joint=LF_crank multiplier=-9
- added joint LF_rotorB: type revolute, parent pod_LF, child rotorB_LF, origin xyz=0.04675 0.00000 0.06000, axis 0 1 0, limit lower=-174.53293 upper=174.53293 effort=3.5 velocity=210, mimic joint=LF_hip multiplier=-9
- added joint LF_rotorC: type revolute, parent torso, child rotorC_LF, origin xyz=0.22150 0.10000 0.02400, axis 1 0 0, limit lower=-174.53293 upper=174.53293 effort=3.5 velocity=210, mimic joint=LF_abad multiplier=-9
- added joint LR_rotorA: type revolute, parent pod_LR, child rotorA_LR, origin xyz=-0.04675 0.00000 0.06000, axis 0 1 0, limit lower=-174.53293 upper=174.53293 effort=3.5 velocity=210, mimic joint=LR_crank multiplier=-9
- added joint LR_rotorB: type revolute, parent pod_LR, child rotorB_LR, origin xyz=0.04675 0.00000 0.06000, axis 0 1 0, limit lower=-174.53293 upper=174.53293 effort=3.5 velocity=210, mimic joint=LR_hip multiplier=-9
- added joint LR_rotorC: type revolute, parent torso, child rotorC_LR, origin xyz=-0.22150 0.10000 0.02400, axis 1 0 0, limit lower=-174.53293 upper=174.53293 effort=3.5 velocity=210, mimic joint=LR_abad multiplier=-9
- added joint RF_rotorA: type revolute, parent pod_RF, child rotorA_RF, origin xyz=-0.04675 0.00000 0.06000, axis 0 1 0, limit lower=-174.53293 upper=174.53293 effort=3.5 velocity=210, mimic joint=RF_crank multiplier=-9
- added joint RF_rotorB: type revolute, parent pod_RF, child rotorB_RF, origin xyz=0.04675 0.00000 0.06000, axis 0 1 0, limit lower=-174.53293 upper=174.53293 effort=3.5 velocity=210, mimic joint=RF_hip multiplier=-9
- added joint RF_rotorC: type revolute, parent torso, child rotorC_RF, origin xyz=0.22150 -0.10000 0.02400, axis 1 0 0, limit lower=-174.53293 upper=174.53293 effort=3.5 velocity=210, mimic joint=RF_abad multiplier=-9
- added joint RR_rotorA: type revolute, parent pod_RR, child rotorA_RR, origin xyz=-0.04675 0.00000 0.06000, axis 0 1 0, limit lower=-174.53293 upper=174.53293 effort=3.5 velocity=210, mimic joint=RR_crank multiplier=-9
- added joint RR_rotorB: type revolute, parent pod_RR, child rotorB_RR, origin xyz=0.04675 0.00000 0.06000, axis 0 1 0, limit lower=-174.53293 upper=174.53293 effort=3.5 velocity=210, mimic joint=RR_hip multiplier=-9
- added joint RR_rotorC: type revolute, parent torso, child rotorC_RR, origin xyz=-0.22150 -0.10000 0.02400, axis 1 0 0, limit lower=-174.53293 upper=174.53293 effort=3.5 velocity=210, mimic joint=RR_abad multiplier=-9
- joint LF_coupler: limit lower=-1.04720 upper=1.04720 effort=31.5 velocity=23.3 -> lower=-1.04720 upper=1.04720 effort=0 velocity=23.3; mimic joint=LF_knee multiplier=-1 -> (none)
- joint LF_crank: limit lower=-1.04720 upper=1.04720 effort=31.5 velocity=23.3 -> lower=-1.57080 upper=1.57080 effort=31.5 velocity=23.3; mimic joint=LF_knee multiplier=1 -> (none); origin xyz=0.00000 0.00000 0.00000 -> xyz=0.00000 0.07950 -0.00979; parent thigh_LF -> pod_LF
- joint LF_knee: limit lower=-1.04720 upper=1.04720 effort=31.5 velocity=23.3 -> lower=-1.04720 upper=1.04720 effort=0 velocity=23.3
- joint LR_coupler: limit lower=-1.04720 upper=1.04720 effort=31.5 velocity=23.3 -> lower=-1.04720 upper=1.04720 effort=0 velocity=23.3; mimic joint=LR_knee multiplier=-1 -> (none)
- joint LR_crank: limit lower=-1.04720 upper=1.04720 effort=31.5 velocity=23.3 -> lower=-1.57080 upper=1.57080 effort=31.5 velocity=23.3; mimic joint=LR_knee multiplier=1 -> (none); origin xyz=0.00000 0.00000 0.00000 -> xyz=0.00000 0.07950 -0.00979; parent thigh_LR -> pod_LR
- joint LR_knee: limit lower=-1.04720 upper=1.04720 effort=31.5 velocity=23.3 -> lower=-1.04720 upper=1.04720 effort=0 velocity=23.3
- joint RF_coupler: limit lower=-1.04720 upper=1.04720 effort=31.5 velocity=23.3 -> lower=-1.04720 upper=1.04720 effort=0 velocity=23.3; mimic joint=RF_knee multiplier=-1 -> (none)
- joint RF_crank: limit lower=-1.04720 upper=1.04720 effort=31.5 velocity=23.3 -> lower=-1.57080 upper=1.57080 effort=31.5 velocity=23.3; mimic joint=RF_knee multiplier=1 -> (none); origin xyz=0.00000 0.00000 0.00000 -> xyz=0.00000 -0.07950 -0.00979; parent thigh_RF -> pod_RF
- joint RF_knee: limit lower=-1.04720 upper=1.04720 effort=31.5 velocity=23.3 -> lower=-1.04720 upper=1.04720 effort=0 velocity=23.3
- joint RR_coupler: limit lower=-1.04720 upper=1.04720 effort=31.5 velocity=23.3 -> lower=-1.04720 upper=1.04720 effort=0 velocity=23.3; mimic joint=RR_knee multiplier=-1 -> (none)
- joint RR_crank: limit lower=-1.04720 upper=1.04720 effort=31.5 velocity=23.3 -> lower=-1.57080 upper=1.57080 effort=31.5 velocity=23.3; mimic joint=RR_knee multiplier=1 -> (none); origin xyz=0.00000 0.00000 0.00000 -> xyz=0.00000 -0.07950 -0.00979; parent thigh_RR -> pod_RR
- joint RR_knee: limit lower=-1.04720 upper=1.04720 effort=31.5 velocity=23.3 -> lower=-1.04720 upper=1.04720 effort=0 velocity=23.3
